Commit message: pointcloud->costmap 변환시에 바닥도 장애물로 표현됨

File: urdf/kobuki_stereo.urdf.xacro (robot description, xacro)
@@ -7,8 +7,7 @@
   <!-- Defines the kobuki component tag. -->
   <xacro:include filename="$(find kobuki_2dnav_sim)/urdf/kobuki.urdf.xacro" />
-  <xacro:include filename="$(find kobuki_2dnav_sim)/urdf/hokuyo.urdf.xacro"/>
-  <!--<xacro:include filename="$(find kobuki_2dnav_sim)/urdf/stereo.urdf.xacro"/>-->
+  <xacro:include filename="$(find kobuki_2dnav_sim)/urdf/stereo.urdf.xacro"/>
   <xacro:sensor_hokuyo name="laser" parent="base_link">
-      <origin xyz="0 0 0.12" rpy="0 0 0"/>
+      <origin xyz="0 0 0.52" rpy="0 0 0"/>
   </xacro:sensor_hokuyo>
   <kobuki/>
